Commit message: 尝试修改小车为烧饼的样子

File: src/bringup/src/description/jiuche.urdf (robot description, URDF)
Before this commit: robot xiaoche, 2 links, 1 joints
Links:
- added link caster_link; collision sphere radius=0.10; visual sphere radius=0.10
Joints:
- added joint caster_joint: type fixed, parent base_link, child caster_link, origin xyz=${base_radius - 0.10} 0 0.05
